Commit message: Tweak Computed Torque parameters, fix URDF values and add ROS2 .gitignore

File: simulation_2dof/urdf/robot_2dof.urdf (robot description, URDF)
Before this commit: robot pendulum_2dof, 4 links, 3 joints
Joints:
- joint joint1: axis 0 1 0 -> 0 0 1; type revolute -> continuous
- joint joint2: axis 0 1 0 -> 0 0 1; type revolute -> continuous

Commit message: feature: kalman filter and plot with rosbag

File: simulation_2dof/urdf/robot_2dof.urdf (robot description, URDF)
Before this commit: robot pendulum_2dof, 4 links, 3 joints
Joints:
- joint joint1: axis 0 1 0 -> 0 0 1
- joint joint2: axis 0 1 0 -> 0 0 1
